Commit message: Modified robot model and added ball movement script

File: urdf/robot.xacro (robot description, xacro)
@@ -40,5 +40,5 @@
     <color rgba="1.0 1.0 1.0 1.0"/>
   </material>
-	  <link name="link_chassis">
+	<link name="link_chassis">
     <!-- pose and inertial -->
     <pose>0 0 0.1 0 0 0</pose>
@@ -51,5 +51,5 @@
     <collision name="collision_chassis">
       <geometry>
-        <box size="0.5 0.3 0.07"/>
+        <box size="0.5 0.3 0.1"/>
       </geometry>
     </collision>
@@ -57,7 +57,7 @@
       <origin rpy="0 0 0" xyz="0 0 0"/>
       <geometry>
-        <box size="0.5 0.3 0.07"/>
+        <box size="0.5 0.3 0.1"/>
       </geometry>
-      <material name="blue"/>
+      <material name="orange"/>
     </visual>
     <!-- caster front -->
@@ -75,5 +75,6 @@
     </visual>
   </link>
-   <link name="link_right_wheel">
+  <!-- wheels -->
+  <link name="link_right_wheel">
     <xacro:default_inertial mass="0.2"/>
     <collision name="link_right_wheel_collision">
@@ -115,19 +116,64 @@
     <joint_properties damping="1.0" friction="1.0"/>
   </joint>
+  <!-- neck and head -->
+  <link name="link_neck">
+    <xacro:default_inertial mass="0.5"/>
+    <collision name="link_neck_collision">
+      <origin rpy="0 0 0" xyz="0.1 0 0.05"/>
+      <geometry>
+        <cylinder length="0.1" radius="0.05"/>
+      </geometry>
+    </collision>
+    <visual name="link_neck_visual">
+      <origin rpy="0 0 0" xyz="0.1 0 0.05"/>
+      <geometry>
+        <cylinder length="0.1" radius="0.05"/>
+      </geometry>
+      <material name="orange"/>
+    </visual>
+  </link>
+  <link name="link_head">
+    <xacro:default_inertial mass="0.5"/>
+    <collision name="link_head_collision">
+      <origin rpy="0 0 0" xyz="0.05 0 0.15"/>
+      <geometry>
+        <box size= "0.15 0.2 0.15"/>
+      </geometry>
+    </collision>
+    <visual name="link_head_visual">
+      <origin rpy="0 0 0" xyz="0.05 0 0.15"/>
+      <geometry>
+        <box size= "0.15 0.2 0.15"/>
+      </geometry>
+      <material name="orange"/>
+    </visual>
+  </link>
+  <joint name="joint_neck" type="fixed">
+    <origin rpy="0 0 0" xyz="0.1 0 0.05"/>
+    <child link="link_neck"/>
+    <parent link="link_chassis"/>
+  </joint>
+  <joint name="joint_head" type="revolute">
+    <origin rpy="0 0 0" xyz="0 0 0"/>
+    <child link="link_head"/>
+    <parent link="link_neck"/>
+    <axis rpy="0 0 1" xyz="0 0 0"/>
+    <limit effort="10000" velocity="1000"/>
+    <joint_properties damping="1.0" friction="1.0"/>
+  </joint>
+  <!-- camera -->
   <link name="camera_link">
 	    <collision>
-	      <origin xyz="0 0 0.025" rpy="0 0 0"/>
+	      <origin xyz="0.125 0 0.1" rpy="0 0 0"/>
 	      <geometry>
-		<box size="0.05 0.05 0.05"/>
+		      <box size="0.05 0.05 0.05"/>
 	      </geometry>
 	    </collision>
 	    <visual>
-	      <origin xyz="0 0 0.025" rpy="0 0 0"/>
+	      <origin xyz="0.125 0 0.1" rpy="0 0 0"/>
 	      <geometry>
-		<box size="0.05 0.05 0.05"/>
+		      <box size="0.05 0.05 0.05"/>
 	      </geometry>
-	      <material name="red">
-		<color rgba="1 0 0 1"/>
-	      </material>
+	      <material name="grey"/>
 	    </visual>
 	    <inertial>
@@ -139,6 +185,6 @@
   <joint name="camera_joint" type="fixed">
 	    <axis xyz="0 1 0" />
-	    <origin xyz="0.23 0 0.0" rpy="0 0 0"/>
-	    <parent link="link_chassis"/>
+	    <origin xyz="0 0 0.0" rpy="0 0 0"/>
+	    <parent link="link_head"/>
 	    <child link="camera_link"/>
 	 </joint>

Commit message: Added Play behaviour and behaviour controller
Some problems in the play behavior movements

File: urdf/robot.xacro (robot description, xacro)
@@ -136,5 +136,5 @@
     <xacro:default_inertial mass="0.5"/>
     <collision name="link_head_collision">
-      <origin rpy="0 0 0" xyz="0.05 0 0.15"/>
+      <origin rpy="0 0 0" xyz="0.15 0 0.15"/>
       <geometry>
         <box size= "0.15 0.2 0.15"/>
@@ -142,5 +142,5 @@
     </collision>
     <visual name="link_head_visual">
-      <origin rpy="0 0 0" xyz="0.05 0 0.15"/>
+      <origin rpy="0 0 0" xyz="0.15 0 0.15"/>
       <geometry>
         <box size= "0.15 0.2 0.15"/>
@@ -150,5 +150,6 @@
   </link>
   <joint name="joint_neck" type="fixed">
-    <origin rpy="0 0 0" xyz="0.1 0 0.05"/>
+    <axis xyz="0 1 0" />
+	  <origin xyz="0.1 0 0.05" rpy="0 0 0"/>
     <child link="link_neck"/>
     <parent link="link_chassis"/>
@@ -165,5 +166,5 @@
   <link name="camera_link">
 	    <collision>
-	      <origin xyz="0.125 0 0.1" rpy="0 0 0"/>
+	      <origin xyz="0.025 0 0.15" rpy="0 0 0"/>
 	      <geometry>
 		      <box size="0.05 0.05 0.05"/>
@@ -171,5 +172,5 @@
 	    </collision>
 	    <visual>
-	      <origin xyz="0.125 0 0.1" rpy="0 0 0"/>
+	      <origin xyz="0.025 0 0.15" rpy="0 0 0"/>
 	      <geometry>
 		      <box size="0.05 0.05 0.05"/>
@@ -185,7 +186,7 @@
   <joint name="camera_joint" type="fixed">
 	    <axis xyz="0 1 0" />
-	    <origin xyz="0 0 0.0" rpy="0 0 0"/>
+	    <origin xyz="0.15 0 0.0" rpy="0 0 0"/>
+      <child link="camera_link"/>
 	    <parent link="link_head"/>
-	    <child link="camera_link"/>
 	 </joint>
 </robot>

Commit message: Added ros_control for joint head position

File: urdf/robot.xacro (robot description, xacro)
@@ -160,5 +160,6 @@
     <parent link="link_neck"/>
     <axis rpy="0 0 1" xyz="0 0 0"/>
-    <limit effort="10000" velocity="1000"/>
+    <limit effort ="1000" lower="0" upper="1000"
+velocity="1000"/>
     <joint_properties damping="1.0" friction="1.0"/>
   </joint>

Commit message: Adjusted robot description for  joint_robot_controller

File: urdf/robot.xacro (robot description, xacro)
@@ -159,7 +159,6 @@
     <child link="link_head"/>
     <parent link="link_neck"/>
-    <axis rpy="0 0 1" xyz="0 0 0"/>
-    <limit effort ="1000" lower="0" upper="1000"
-velocity="1000"/>
+    <axis xyz="0 0 1"/>
+    <limit effort="1000.0" lower="-1.57" upper="1.57" velocity="0.2"/>/>
     <joint_properties damping="1.0" friction="1.0"/>
   </joint>
@@ -190,4 +189,14 @@
       <child link="camera_link"/>
 	    <parent link="link_head"/>
-	 </joint>
+	</joint>
+  <transmission name="joint_head_trans">
+	  <type>transmission_interface/SimpleTransmission</type>
+	  <joint name="joint_head">
+		<hardwareInterface>hardware_interface/EffortJointInterface</hardwareInterface>
+	</joint>
+	<actuator name="motor1">
+		<hardwareInterface>hardware_interface/EffortJointInterface</hardwareInterface>
+		<mechanicalInterface>1</mechanicalInterface>
+	</actuator>
+  </transmission>
 </robot>

Commit message: Adjusted head moving

File: urdf/robot.xacro (robot description, xacro)
@@ -160,5 +160,5 @@
     <parent link="link_neck"/>
     <axis xyz="0 0 1"/>
-    <limit effort="1000.0" lower="-1.57" upper="1.57" velocity="0.2"/>/>
+    <limit effort="1000.0" lower="-1.57" upper="1.57" velocity="0.1"/>/>
     <joint_properties damping="1.0" friction="1.0"/>
   </joint>
